File: kicad/adc_clk.kicad_sch (KiCad schematic)
At the start: 39 parts, among them U8 AD9649BCPZ-80, U9 LMK61E2-100M00SIAR

Commit message: Bus pin swap, FT601 IO registers, ADC clock layout, working board and fan-out tooling
- FPGA ball re-assignment (AGY, verified): FT601 and ADC buses planar; LPF, design.py, schematic, netlist synced.
- Gateware: FT601 outputs/tristates in IOLOGIC on a +112.5 deg PLL clock; AD9649 DCO inverted at boot.
- ADC sample clock laid out on F.Cu with swapped polarity; BOM U9 corrected to the 8-pin I2C LMK61E2.
- kicad/work: DeepPCB run 2 board plus scripted patches (buck, In2 GND fill, VCCAUX, clock); DeepPCB snapshots.
- kicad/gen: patch, repair, routing and fan-out scripts (fanout_apply, fanout_trial, place_free, escape_apply).
- notes/pinswap, notes/fanout: briefs, AGY results and Claude's reviews.
- Vendor datasheets removed from the repo; refs/datasheets.md lists their sources.

Co-Authored-By: Claude Opus 5.5 <noreply@anthropic.com>
Connections:
- net ADC_CLKN: now also C61.2; no longer C62.2
- net ADC_CLKP: now also C62.2; no longer C61.2
